File: PCB/BasisStation/JTAG-PROG.kicad_sch (KiCad schematic)
At the start: 4 parts, among them X2 JTAG

Commit message: Schaltplan angepasst
Parts:
- C3, C6: value 100µF -> 100nF
Changed lines of the file:
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@@
 			)
 		)
-		(property "Value" "100µF"
+		(property "Value" "100nF"
 			(at 133.35 65.1509 0)
 			(effects
@@
 			)
 		)
-		(property "Value" "100µF"
+		(property "Value" "100nF"
 			(at 133.35 131.1909 0)
 			(effects

Commit message: neue Bauteile hinzugefügt
Changed lines of the file:
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@@
 		(property "Value" "100nF"
 			(at 133.35 65.1509 0)
+			(show_name yes)
 			(effects
 				(font
