File: PCB/BasisStation/BasisStation.kicad_pcb (KiCad board)
At the start: 2 copper layers, 150 x 113.5 mm, 21 parts, among them SW1 SW_SPST, SW4 RESET_BUTTON, U1 ESP32-S3-WROOM-1-N16R8, X2 JTAG

Commit message: Backups gelöscht
Parts:
- removed C2: 100µF, CUSTOM_Footprint:CAPAE1030X1050N
- C1: value 4700µF -> 100µF
- moved C1 72.5 mm to (115.2, 82.5)
- moved R5 4.60 mm to (104.5, 76.9)
Connections:
- C1 pad P: (no net) -> +3.3V
Routing:
- net +3.3V: track 345.1 -> 358.1 mm
- net Boot Mode: track 45.5 -> 34.7 mm
- net 3,3V: track 40.4 -> 35.8 mm
- net GND: track 0.50 -> 2.50 mm, vias 0 -> 1
