File: PCB/BasisStation/BasisStation.kicad_sch (KiCad schematic)
At the start: 19 parts, among them SW3 SW_SPST, SW4 RESET_BUTTON, U2 ESP32-S3-WROOM-2, X4 JTAG

Commit message: Backups gelöscht
Parts:
- removed C1: 100µF, CUSTOM_Footprint:CAPAE1030X1050N, symbol Device:C_Polarized
Connections:
- net 27: no longer names the net of U2.27 (GPIO0/BOOT), X3.6 (Pin_6)
Changed lines of the file:
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@@
 	(wire
 		(pts
-			(xy 26.67 276.86) (xy 26.67 279.4)
+			(xy 27.94 274.32) (xy 27.94 276.86)
 		)
 		(stroke
@@
 	(wire
 		(pts
-			(xy 36.83 276.86) (xy 36.83 279.4)
+			(xy 38.1 274.32) (xy 38.1 276.86)
 		)
 		(stroke
@@
 	(wire
 		(pts
-			(xy 16.51 276.86) (xy 16.51 279.4)
+			(xy 17.78 274.32) (xy 17.78 276.86)
 		)
 		(stroke
@@
 		)
 	)
-	(label "27"
-		(at 181.61 74.93 0)
-		(fields_autoplaced yes)
-		(effects
-			(font
-				(size 1.27 1.27)
-			)
-			(justify left bottom)
-		)
-	)
 	(label "EN"
 		(at 160.02 69.85 0)
@@
 	(symbol
 		(lib_id "power:PWR_FLAG")
-		(at 36.83 276.86 0)
+		(at 38.1 274.32 0)
 		(unit 1)
 		(exclude_from_sim no)
@@
 		(fields_autoplaced yes)
 		(property "Reference" "#FLG02"
-			(at 36.83 274.955 0)
+			(at 38.1 272.415 0)
 			(effects
 				(font
@@
 		)
 		(property "Value" "PWR_FLAG"
-			(at 36.83 271.78 0)
+			(at 38.1 269.24 0)
 			(effects
 				(font
@@
 		)
 		(property "Footprint" ""
-			(at 36.83 276.86 0)
+			(at 38.1 274.32 0)
 			(effects
 				(font
@@
 		)
 		(property "Datasheet" "~"
-			(at 36.83 276.86 0)
+			(at 38.1 274.32 0)
 			(effects
 				(font
@@
 		)
 		(property "Description" "Special symbol for telling ERC where power comes from"
-			(at 36.83 276.86 0)
+			(at 38.1 274.32 0)
 			(effects
 				(font
@@
 	)
 	(symbol
-		(lib_id "Device:C_Polarized")
-		(at 73.66 63.5 0)
-		(unit 1)
-		(exclude_from_sim no)
-		(in_bom yes)
-		(on_board yes)
-		(dnp no)
-		(fields_autoplaced yes)
-		(property "Reference" "C1"
-			(at 77.47 61.3409 0)
-			(effects
-				(font
-					(size 1.27 1.27)
-				)
-				(justify left)
-			)
-		)
-		(property "Value" "100µF"
-			(at 77.47 63.8809 0)
-			(effects
-				(font
-					(size 1.27 1.27)
-				)
-				(justify left)
-			)
-		)
-		(property "Footprint" "CUSTOM_Footprint:CAPAE1030X1050N"
-			(at 74.6252 67.31 0)
-			(effects
-				(font
-					(size 1.27 1.27)
-				)
-				(hide yes)
-			)
-		)
-		(property "Datasheet" "chrome-extension://efaidnbmnnnibpcajpcglclefindmkaj/https://www.we-online.com/components/products/datasheet/865060343005.pdf"
-			(at 73.66 63.5 0)
-			(effects
-				(font
-					(size 1.27 1.27)
-				)
-				(hide yes)
-			)
-		)
-		(property "Description" "Polarized capacitor"
-			(at 73.66 63.5 0)
-			(effects
-				(font
-					(size 1.27 1.27)
-				)
-				(hide yes)
-			)
-		)
-		(pin "2"
-		)
-		(pin "1"
-		)
-		(instances
-			(project "BasisStation"
-				(path "/cc03a18a-a128-4e00-a998-441923eeacd1"
-					(reference "C1")
-					(unit 1)
-				)
-			)
-		)
-	)
-	(symbol
 		(lib_id "PCM_Espressif:ESP32-S3-WROOM-2")
 		(at 105.41 133.35 0)
@@
 	(symbol
 		(lib_id "power:PWR_FLAG")
-		(at 26.67 276.86 0)
+		(at 27.94 274.32 0)
 		(unit 1)
 		(exclude_from_sim no)
@@
 		(fields_autoplaced yes)
 		(property "Reference" "#FLG03"
-			(at 26.67 274.955 0)
+			(at 27.94 272.415 0)
 			(effects
 				(font
@@
 		)
 		(property "Value" "PWR_FLAG"
-			(at 26.67 271.78 0)
+			(at 27.94 269.24 0)
 			(effects
 				(font
@@
 		)
 		(property "Footprint" ""
-			(at 26.67 276.86 0)
+			(at 27.94 274.32 0)
 			(effects
 				(font
@@
 		)
 		(property "Datasheet" "~"
-			(at 26.67 276.86 0)
+			(at 27.94 274.32 0)
 			(effects
 				(font
@@
 		)
 		(property "Description" "Special symbol for telling ERC where power comes from"
-			(at 26.67 276.86 0)
+			(at 27.94 274.32 0)
 			(effects
 				(font
@@
 	(symbol
 		(lib_id "power:VCC")
-		(at 26.67 279.4 180)
+		(at 27.94 276.86 180)
 		(unit 1)
 		(exclude_from_sim no)
@@
 		(fields_autoplaced yes)
 		(property "Reference" "#PWR017"
-			(at 26.67 275.59 0)
+			(at 27.94 273.05 0)
 			(effects
 				(font
@@
 		)
 		(property "Value" "+3.3V"
-			(at 26.67 284.48 0)
+			(at 27.94 281.94 0)
 			(effects
 				(font
@@
 		)
 		(property "Footprint" ""
-			(at 26.67 279.4 0)
+			(at 27.94 276.86 0)
 			(effects
 				(font
@@
 		)
 		(property "Datasheet" ""
-			(at 26.67 279.4 0)
+			(at 27.94 276.86 0)
 			(effects
 				(font
@@
 		)
 		(property "Description" "Power symbol creates a global label with name \"VCC\""
-			(at 26.67 279.4 0)
+			(at 27.94 276.86 0)
 			(effects
 				(font
@@
 	(symbol
 		(lib_id "power:GND")
-		(at 36.83 279.4 0)
+		(at 38.1 276.86 0)
 		(unit 1)
 		(exclude_from_sim no)
@@
 		(fields_autoplaced yes)
 		(property "Reference" "#PWR016"
-			(at 36.83 285.75 0)
+			(at 38.1 283.21 0)
 			(effects
 				(font
@@
 		)
 		(property "Value" "GND"
-			(at 36.83 284.48 0)
+			(at 38.1 281.94 0)
 			(effects
 				(font
@@
 		)
 		(property "Footprint" ""
-			(at 36.83 279.4 0)
+			(at 38.1 276.86 0)
 			(effects
 				(font
@@
 		)
 		(property "Datasheet" ""
-			(at 36.83 279.4 0)
+			(at 38.1 276.86 0)
 			(effects
 				(font
@@
 		)
 		(property "Description" "Power symbol creates a global label with name \"GND\" , ground"
-			(at 36.83 279.4 0)
+			(at 38.1 276.86 0)
 			(effects
 				(font
@@
 	(symbol
 		(lib_id "power:VCC")
-		(at 16.51 279.4 180)
+		(at 17.78 276.86 180)
 		(unit 1)
 		(exclude_from_sim no)
@@
 		(fields_autoplaced yes)
 		(property "Reference" "#PWR015"
-			(at 16.51 275.59 0)
+			(at 17.78 273.05 0)
 			(effects
 				(font
@@
 		)
 		(property "Value" "+12V"
-			(at 16.51 284.48 0)
+			(at 17.78 281.94 0)
 			(effects
 				(font
@@
 		)
 		(property "Footprint" ""
-			(at 16.51 279.4 0)
+			(at 17.78 276.86 0)
 			(effects
 				(font
@@
 		)
 		(property "Datasheet" ""
-			(at 16.51 279.4 0)
+			(at 17.78 276.86 0)
 			(effects
 				(font
@@
 		)
 		(property "Description" "Power symbol creates a global label with name \"VCC\""
-			(at 16.51 279.4 0)
+			(at 17.78 276.86 0)
 			(effects
 				(font
@@
 	(symbol
 		(lib_id "power:PWR_FLAG")
-		(at 16.51 276.86 0)
+		(at 17.78 274.32 0)
 		(unit 1)
 		(exclude_from_sim no)
@@
 		(fields_autoplaced yes)
 		(property "Reference" "#FLG01"
-			(at 16.51 274.955 0)
+			(at 17.78 272.415 0)
 			(effects
 				(font
@@
 		)
 		(property "Value" "PWR_FLAG"
-			(at 16.51 271.78 0)
+			(at 17.78 269.24 0)
 			(effects
 				(font
@@
 		)
 		(property "Footprint" ""
-			(at 16.51 276.86 0)
+			(at 17.78 274.32 0)
 			(effects
 				(font
@@
 		)
 		(property "Datasheet" "~"
-			(at 16.51 276.86 0)
+			(at 17.78 274.32 0)
 			(effects
 				(font
@@
 		)
 		(property "Description" "Special symbol for telling ERC where power comes from"
-			(at 16.51 276.86 0)
+			(at 17.78 274.32 0)
 			(effects
 				(font
