File: PCB/BasisStation/BasisStation_architektur.kicad_sch (KiCad schematic)
At the start: 0 parts

Commit message: usb-schnittstelle hinzugefügt
Other:
- removed sheet Debugging
- removed sheet Layout
Changed lines of the file:
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@@
 	)
 	(image
-		(at 134.62 95.25)
+		(at 149.86 92.71)
 		(scale 2.72729)
 		(data "iVBORw0KGgoAAAANSUhEUgAAAvkAAAKfCAYAAAD0Edc/AAAAAXNSR0IArs4c6QAAZBN0RVh0bXhm"
@@
 		)
 	)
-	(sheet
-		(at 302.26 0)
-		(size 295.91 210.82)
-		(fields_autoplaced yes)
-		(stroke
-			(width 0.1524)
-			(type solid)
-		)
-		(fill
-			(color 0 0 0 0.0000)
-		)
-		(property "Sheetname" "Layout"
-			(at 302.26 -0.7116 0)
-			(effects
-				(font
-					(size 1.27 1.27)
-				)
-				(justify left bottom)
-			)
-		)
-		(property "Sheetfile" "BasisStation_Layout.kicad_sch"
-			(at 302.26 211.4046 0)
-			(effects
-				(font
-					(size 1.27 1.27)
-				)
-				(justify left top)
-			)
-		)
-		(instances
-			(project "BasisStation"
-				(path "/498c7092-55c1-4229-9f4b-13c6a8e7da47"
-					(page "2")
-				)
-			)
-		)
-	)
-	(sheet
-		(at 1.27 224.79)
-		(size 295.91 152.4)
-		(fields_autoplaced yes)
-		(stroke
-			(width 0.1524)
-			(type solid)
-		)
-		(fill
-			(color 0 0 0 0.0000)
-		)
-		(property "Sheetname" "Debugging"
-			(at 1.27 224.0784 0)
-			(effects
-				(font
-					(size 1.27 1.27)
-				)
-				(justify left bottom)
-			)
-		)
-		(property "Sheetfile" "BasisStation_Debugging.kicad_sch"
-			(at 1.27 377.7746 0)
-			(effects
-				(font
-					(size 1.27 1.27)
-				)
-				(justify left top)
-			)
-		)
-		(instances
-			(project "BasisStation"
-				(path "/498c7092-55c1-4229-9f4b-13c6a8e7da47"
-					(page "3")
-				)
-			)
-		)
-	)
-	(sheet_instances
-		(path "/"
-			(page "1")
-		)
-	)
