File: pcb/BasisStation/BasisStation_Layout.kicad_sch (KiCad schematic)
At the start: 23 parts, among them J5 Conn_02x05_Odd_Even, J6 Conn_02x03_Odd_Even, Q1 BC337, Q2 BC337, Q3 BC337, Q4 BC337, U6 ESP32-S3-WROOM-1U-N16R8

Commit message: v0.00.001 chore(SHBS-4): Symbole aus Bibliothek aktualisiert
KiCad-Lauf "Symbole aus Bibliothek aktualisieren" (Bediener): die zuvor per
Text-Edit erzeugte power:+3V3-Cache-Definition wurde durch das
Bibliotheksoriginal ersetzt (abweichende Referenz-Position, Pfeil aus zwei
Polylines), lib_symbols alphabetisch sortiert.

Laut report.txt aktualisieren #PWR100-#PWR102 (power:+3V3), PS1
(shbs_power:MP2359DJ) und J_PWR1 (shbs_power:USB_C_Receptacle_Power)
fehlerfrei - die Bibliotheksentkopplung aus da60c97 traegt.

ERC: 29 -> 14 Meldungen (4 Fehler, 10 Warnungen). Die verbleibenden Fehler
sind ausschliesslich power_pin_not_driven an U6.2, PS1.5, J_PWR1.A4 und
#PWR100 und haengen an PWR_FLAG/Buck-Topologie (SHBS-4 offen).

Co-Authored-By: Claude Opus 5 <noreply@anthropic.com>
Parts:
- U6: footprint RF_Module:ESP32-S3-WROOM-1U -> Footprints:ESP32-S3-WROOM-1U
Changed lines of the file:
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@@
 	(wire
 		(pts
+			(xy 66.04 22.86) (xy 66.04 25.4)
+		)
+		(stroke
+			(width 0)
+			(type default)
+		)
+	)
+	(wire
+		(pts
 			(xy 86.36 83.82) (xy 86.36 92.71)
 		)
@@
 	(wire
 		(pts
-			(xy 66.04 22.86) (xy 66.04 25.4)
-		)
-		(stroke
-			(width 0)
-			(type default)
-		)
-	)
-	(wire
-		(pts
 			(xy 66.04 22.86) (xy 101.6 22.86)
 		)
@@
 		)
 	)
-	(symbol
-		(lib_id "power:+3V3")
-		(at 270.51 77.47 270)
-		(unit 1)
-		(exclude_from_sim no)
-		(in_bom yes)
-		(on_board yes)
-		(dnp no)
-		(fields_autoplaced yes)
-		(property "Reference" "#PWR101"
-			(at 270.51 71.12 0)
-			(effects
-				(font
-					(size 1.27 1.27)
-				)
-				(hide yes)
-			)
-		)
-		(property "Value" "+3V3"
-			(at 270.51 73.914 0)
-			(effects
-				(font
-					(size 1.27 1.27)
-				)
-			)
-		)
-		(property "Footprint" ""
-			(at 270.51 77.47 0)
-			(effects
-				(font
-					(size 1.27 1.27)
-				)
-				(hide yes)
-			)
-		)
-		(property "Datasheet" ""
-			(at 270.51 77.47 0)
-			(effects
-				(font
-					(size 1.27 1.27)
-				)
-				(hide yes)
-			)
-		)
-		(property "Description" "Power symbol creates a global label with name \"+3V3\""
-			(at 270.51 77.47 0)
-			(effects
-				(font
-					(size 1.27 1.27)
-				)
-				(hide yes)
-			)
-		)
-		(pin "1"
-		)
-		(instances
-			(project "BasisStation"
-				(path "/498c7092-55c1-4229-9f4b-13c6a8e7da47/1af2eb5e-14cd-443f-ae96-dbfda52b298f"
-					(reference "#PWR101")
-					(unit 1)
-				)
-			)
-		)
-	)
 	(label "EN"
 		(at 92.71 53.34 0)
@@
 		)
 	)
-	(symbol
-		(lib_id "power:+3V3")
-		(at 34.29 92.71 0)
-		(unit 1)
-		(exclude_from_sim no)
-		(in_bom yes)
-		(on_board yes)
-		(dnp no)
-		(fields_autoplaced yes)
-		(property "Reference" "#PWR102"
-			(at 34.29 86.36 0)
-			(effects
-				(font
-					(size 1.27 1.27)
-				)
-				(hide yes)
-			)
-		)
-		(property "Value" "+3V3"
-			(at 34.29 89.154 0)
-			(effects
-				(font
-					(size 1.27 1.27)
-				)
-			)
-		)
-		(property "Footprint" ""
-			(at 34.29 92.71 0)
-			(effects
-				(font
-					(size 1.27 1.27)
-				)
-				(hide yes)
-			)
-		)
-		(property "Datasheet" ""
-			(at 34.29 92.71 0)
-			(effects
-				(font
-					(size 1.27 1.27)
-				)
-				(hide yes)
-			)
-		)
-		(property "Description" "Power symbol creates a global label with name \"+3V3\""
-			(at 34.29 92.71 0)
-			(effects
-				(font
-					(size 1.27 1.27)
-				)
-				(hide yes)
-			)
-		)
-		(pin "1"
-		)
-		(instances
-			(project "BasisStation"
-				(path "/498c7092-55c1-4229-9f4b-13c6a8e7da47/1af2eb5e-14cd-443f-ae96-dbfda52b298f"
-					(reference "#PWR102")
-					(unit 1)
-				)
-			)
-		)
-	)
 	(global_label "USB-"
 		(shape input)
@@
 			)
 		)
+		(property "Sim.Pins" "1=K 2=A"
+			(at 254 96.52 0)
+			(effects
+				(font
+					(size 1.27 1.27)
+				)
+				(hide yes)
+			)
+		)
 		(pin "2"
 		)
@@
 			)
 		)
+		(property "Sim.Pins" "1=K 2=A"
+			(at 254 116.84 0)
+			(effects
+				(font
+					(size 1.27 1.27)
+				)
+				(hide yes)
+			)
+		)
 		(pin "1"
 		)
@@
 			)
 		)
+		(property "Sim.Pins" "1=K 2=A"
+			(at 254 106.68 0)
+			(effects
+				(font
+					(size 1.27 1.27)
+				)
+				(hide yes)
+			)
+		)
 		(pin "2"
 		)
@@
 			)
 		)
-		(property "Footprint" "RF_Module:ESP32-S3-WROOM-1U"
+		(property "Footprint" "Footprints:ESP32-S3-WROOM-1U"
 			(at 140.97 144.78 0)
 			(effects
@@
 	)
 	(symbol
+		(lib_id "power:+3V3")
+		(at 270.51 77.47 270)
+		(unit 1)
+		(exclude_from_sim no)
+		(in_bom yes)
+		(on_board yes)
+		(dnp no)
+		(fields_autoplaced yes)
+		(property "Reference" "#PWR101"
+			(at 270.51 71.12 0)
+			(effects
+				(font
+					(size 1.27 1.27)
+				)
+				(hide yes)
+			)
+		)
+		(property "Value" "+3V3"
+			(at 270.51 73.914 0)
+			(effects
+				(font
+					(size 1.27 1.27)
+				)
+			)
+		)
+		(property "Footprint" ""
+			(at 270.51 77.47 0)
+			(effects
+				(font
+					(size 1.27 1.27)
+				)
+				(hide yes)
+			)
+		)
+		(property "Datasheet" ""
+			(at 270.51 77.47 0)
+			(effects
+				(font
+					(size 1.27 1.27)
+				)
+				(hide yes)
+			)
+		)
+		(property "Description" "Power symbol creates a global label with name \"+3V3\""
+			(at 270.51 77.47 0)
+			(effects
+				(font
+					(size 1.27 1.27)
+				)
+				(hide yes)
+			)
+		)
+		(pin "1"
+		)
+		(instances
+			(project "BasisStation"
+				(path "/498c7092-55c1-4229-9f4b-13c6a8e7da47/1af2eb5e-14cd-443f-ae96-dbfda52b298f"
+					(reference "#PWR101")
+					(unit 1)
+				)
+			)
+		)
+	)
+	(symbol
 		(lib_id "Connector_Generic:Conn_02x05_Odd_Even")
 		(at 46.99 97.79 0)
@@
 					(unit 1)
 				)
+			)
+		)
+	)
+	(symbol
+		(lib_id "power:+3V3")
+		(at 34.29 92.71 0)
+		(unit 1)
+		(exclude_from_sim no)
+		(in_bom yes)
+		(on_board yes)
+		(dnp no)
+		(fields_autoplaced yes)
+		(property "Reference" "#PWR102"
+			(at 34.29 86.36 0)
+			(effects
+				(font
+					(size 1.27 1.27)
+				)
+				(hide yes)
+			)
+		)
+		(property "Value" "+3V3"
+			(at 34.29 89.154 0)
+			(effects
+				(font
+					(size 1.27 1.27)
+				)
+			)
+		)
+		(property "Footprint" ""
+			(at 34.29 92.71 0)
+			(effects
+				(font
+					(size 1.27 1.27)
+				)
+				(hide yes)
+			)
+		)
+		(property "Datasheet" ""
+			(at 34.29 92.71 0)
+			(effects
+				(font
+					(size 1.27 1.27)
+				)
+				(hide yes)
+			)
+		)
+		(property "Description" "Power symbol creates a global label with name \"+3V3\""
+			(at 34.29 92.71 0)
+			(effects
+				(font
+					(size 1.27 1.27)
+				)
+				(hide yes)
+			)
+		)
+		(pin "1"
+		)
+		(instances
+			(project "BasisStation"
+				(path "/498c7092-55c1-4229-9f4b-13c6a8e7da47/1af2eb5e-14cd-443f-ae96-dbfda52b298f"
+					(reference "#PWR102")
+					(unit 1)
+				)

Commit message: v0.00.001 fix(SHBS-4): shbs_power wiederhergestellt, +3V3 auf U6-Schiene
Zwei Ursachen, die der ERC-Lauf vom 2026-09-15 offengelegt hat.

sym-lib-table: Der Merge d7a21e2 hat (name "shbs_power") wieder auf
(name "power") zurueckgesetzt und damit die Entkopplung von der
KiCad-Standardbibliothek rueckgaengig gemacht. Folge: power:GND (28x),
power:+3V3 und power:PWR_FLAG nicht aufloesbar, shbs_power unbekannt fuer
PS1 und J_PWR1. Zusaetzlich waren WCAP-FTXX_P10, WCAP-PT5H_6.3X5.2,
WL-TMRC_3MM und 1543-650-149 nie als Symbolbibliotheken registriert.
Zusammen 42 der 46 Warnungen.

BasisStation_Layout.kicad_sch: Das Netz an U6 Pin 2 (C8.1, C10.1, C12.1,
R9.1, J6.2, U6.2 - 15 Draehte) trug weder Label noch Power-Symbol und war
damit ein eigenes, unbenanntes Netz. Der frueheren +3V3-Korrektur lagen
mit #PWR101 und #PWR102 zwei andere 3,3-V-Inseln zugrunde, nicht die
Schiene von U6. #PWR103 am zuvor offenen Drahtende (248,92 / 22,86)
schliesst sie an und loest zugleich eine unconnected_wire_endpoint-Warnung.
Dieser Drahtstummel darf daher nicht mehr geloescht werden.

ERC-Lauf 2026-09-15 21:43: Meldungen 48 -> 10, Fehler 2 -> 1,
Warnungen 46 -> 9.

Co-Authored-By: Claude Opus 5 <noreply@anthropic.com>
Connections:
- net +3V3: now also C10.1, C12.1, C8.1, J6.2 (Pin_2), R9.1, U6.2 (3V3)
Changed lines of the file:
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@@
+		)
+	)
+	(symbol
+		(lib_id "power:+3V3")
+		(at 248.92 22.86 0)
+		(unit 1)
+		(exclude_from_sim no)
+		(in_bom yes)
+		(on_board yes)
+		(dnp no)
+		(fields_autoplaced yes)
+		(property "Reference" "#PWR103"
+			(at 248.92 16.509999999999998 0)
+			(effects
+				(font
+					(size 1.27 1.27)
+				)
+				(hide yes)
+			)
+		)
+		(property "Value" "+3V3"
+			(at 248.92 19.304 0)
+			(effects
+				(font
+					(size 1.27 1.27)
+				)
+			)
+		)
+		(property "Footprint" ""
+			(at 248.92 22.86 0)
+			(effects
+				(font
+					(size 1.27 1.27)
+				)
+				(hide yes)
+			)
+		)
+		(property "Datasheet" ""
+			(at 248.92 22.86 0)
+			(effects
+				(font
+					(size 1.27 1.27)
+				)
+				(hide yes)
+			)
+		)
+		(property "Description" "Power symbol creates a global label with name \"+3V3\""
+			(at 248.92 22.86 0)
+			(effects
+				(font
+					(size 1.27 1.27)
+				)
+				(hide yes)
+			)
+		)
+		(pin "1"
+		)
+		(instances
+			(project "BasisStation"
+				(path "/498c7092-55c1-4229-9f4b-13c6a8e7da47/1af2eb5e-14cd-443f-ae96-dbfda52b298f"
+					(reference "#PWR103")
+					(unit 1)
+				)
+			)
 		)
 	)
