File: pcb/BasisStation/BasisStation_Layout.kicad_sch (KiCad schematic)
At the start: 26 parts, among them J6 Conn_02x03_Odd_Even, Q1 BC337, Q2 BC337, Q3 BC337, Q4 BC337, U6 ESP32-S3-WROOM-1U-N16R8

Commit message: v0.00.001 fix(SHBS-16): ANT2 auf Seriennachfolger GW.20.A151 umgestellt
Taoglas GW.20.5150 ist abgekuendigt - der Typ steht nicht mehr im
Taoglas-Katalog. Ersetzt durch den Seriennachfolger GW.20.A151: form-,
anschluss- und gewinngleich (2 dBi, 2,4 GHz, RP-SMA(M) gerade).

Zusaetzlich ist Taoglas bei Mouser auf das 960er-Praefix umgezogen, die
alten 742er-Nummern liefern keinen Treffer mehr. Sechs Felder in
BasisStation_Layout.kicad_sch:

- ANT2 Value und Manufacturer_Part_Number: GW.20.5150 -> GW.20.A151
- ANT2 Mouser Part Number: 742-GW.20.5150 -> 960-GW.20.A151
- ANT1 Mouser Part Number: 742-CAB.6061 -> 960-CAB.6061
- beide Produktlinks auf die aktuellen Seiten

Kein Footprint betroffen: ANT1 und ANT2 sind mit on_board no als reine
BOM-Eintraege gefuehrt und kommen nicht auf die Leiterplatte. Mechanisch
bleibt alles gleich, die SMA-Bohrung richtet sich weiter nach dem Pigtail.

Geaendert wurden ausschliesslich Property-Werte - weder lib_id noch
Geometrie beruehrt, daher kein Symbol-Cache-Thema.

Validiert: ERC 0 Verstoesse (0 Fehler, 0 Warnungen). Stueckliste neu
erzeugt, beide Antennen jetzt Status "eindeutig", 16 statt 15 Positionen
mit Preis, LibreOffice rechnet fehlerfrei durch.

Keine Versionserhoehung - kein ESP32-Quellcode geaendert.

Co-Authored-By: Claude Opus 5 <noreply@anthropic.com>
Parts:
- ANT1: Mouser Part Number 742-CAB.6061 -> 960-CAB.6061; Mouser Price/Stock https://www.mouser.de/ProductDetail/Taoglas/CAB-6061 -> https://www.mouser.de/de/ProductDetail/Taoglas/CAB.6061
- ANT2: value GW.20.5150 -> GW.20.A151; Manufacturer_Part_Number GW.20.5150 -> GW.20.A151; Mouser Part Number 742-GW.20.5150 -> 960-GW.20.A151; Mouser Price/Stock https://www.mouser.de/ProductDetail/Taoglas/GW-20-5150 -> https://www.mouser.de/de/ProductDetail/Taoglas/GW.20.A151
Changed lines of the file:
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@@
 			)
 		)
-		(property "Value" "GW.20.5150"
+		(property "Value" "GW.20.A151"
 			(at 149.86 147.3199 0)
 			(effects
@@
 			)
 		)
-		(property "Manufacturer_Part_Number" "GW.20.5150"
-			(at 135.89 146.05 0)
-			(effects
-				(font
-					(size 1.27 1.27)
-				)
-				(hide yes)
-			)
-		)
-		(property "Mouser Part Number" "742-GW.20.5150"
-			(at 135.89 146.05 0)
-			(effects
-				(font
-					(size 1.27 1.27)
-				)
-				(hide yes)
-			)
-		)
-		(property "Mouser Price/Stock" "https://www.mouser.de/ProductDetail/Taoglas/GW-20-5150"
+		(property "Manufacturer_Part_Number" "GW.20.A151"
+			(at 135.89 146.05 0)
+			(effects
+				(font
+					(size 1.27 1.27)
+				)
+				(hide yes)
+			)
+		)
+		(property "Mouser Part Number" "960-GW.20.A151"
+			(at 135.89 146.05 0)
+			(effects
+				(font
+					(size 1.27 1.27)
+				)
+				(hide yes)
+			)
+		)
+		(property "Mouser Price/Stock" "https://www.mouser.de/de/ProductDetail/Taoglas/GW.20.A151"
 			(at 135.89 146.05 0)
 			(effects
@@
 			)
 		)
-		(property "Mouser Part Number" "742-CAB.6061"
-			(at 74.93 147.32 0)
-			(effects
-				(font
-					(size 1.27 1.27)
-				)
-				(hide yes)
-			)
-		)
-		(property "Mouser Price/Stock" "https://www.mouser.de/ProductDetail/Taoglas/CAB-6061"
-			(at 74.93 147.32 0)
-			(effects
+		(property "Mouser Part Number" "960-CAB.6061"
+			(at 74.93 147.32 0)
+			(effects
+				(font
+					(size 1.27 1.27)
+				)
+				(hide yes)
+			)
+		)
+		(property "Mouser Price/Stock" "https://www.mouser.de/de/ProductDetail/Taoglas/CAB.6061"
+			(at 74.93 147.32 0)
+			(effects

Commit message: v0.00.001 feat(SHBS-17): Teilenummern fuer 29 Positionen in den Schaltplan uebernommen
Die vom Bediener freigegebenen Teilevorschlaege (Hausstandard Passivteile, LEDs, Q1-Q4, F1, FB1) stehen jetzt als Felder Manufacturer, Manufacturer_Part_Number und Mouser Part Number an 58 Instanzen. F1-Wert von Fuse auf 1.1A gesetzt. Gegenprobe: keine Felder verloren, Netzliste identisch (102 Netze), ERC 0 Fehler.

Stueckliste gruppiert jetzt nach Herstellerteilenummer (Werte sind uneinheitlich geschrieben): 44 Positionen, alle lieferbar, 47,78 EUR. PROPOSED_PARTS geleert, Hausstandard in hardware.md dokumentiert, Bestellteile in power_supply.md aktualisiert.

Co-Authored-By: Claude Opus 5.5 <noreply@anthropic.com>
Parts:
- D10: Manufacturer (none) -> Würth Elektronik; Manufacturer_Part_Number (none) -> 151031VS06000; Mouser Part Number (none) -> 710-151031VS06000
- D8: Manufacturer (none) -> Würth Elektronik; Manufacturer_Part_Number (none) -> 151033BS03000; Mouser Part Number (none) -> 710-151033BS03000
- D9: Manufacturer (none) -> Würth Elektronik; Manufacturer_Part_Number (none) -> 151033RS03000; Mouser Part Number (none) -> 710-151033RS03000
- Q1, Q2, Q3, Q4: Manufacturer (none) -> onsemi; Manufacturer_Part_Number (none) -> BC33740TA; Mouser Part Number (none) -> 512-BC33740TA
- R13, R14, R15, R16: Manufacturer (none) -> Vishay BC Components; Manufacturer_Part_Number (none) -> PR02000202200JR500; Mouser Part Number (none) -> 594-5083NW220R0J
- R23, R24, R25, R26: Manufacturer (none) -> Vishay BC Components; Manufacturer_Part_Number (none) -> PR02000204701JR500; Mouser Part Number (none) -> 594-5083NW4K700J
- R9: Manufacturer (none) -> YAGEO; Manufacturer_Part_Number (none) -> MFR-25FBF52-10K; Mouser Part Number (none) -> 603-MFR-25FBF52-10K

Commit message: v0.00.001 feat(SHBS-17): Abgeleitete Teilenummern bestaetigt und eingetragen, SHBS-17 abgeschlossen
D11 Comchip SS34-HF (SMA; die guenstigere Slkormicro-SS34 ist SMC und passt nicht auf D_SMA), D12 Littelfuse SMAJ5.0A, U1 D3V3XA4B10LP-7, L1 Bourns SRN6045TA-100M, J6 Wuerth 61200621621 als Felder im Schaltplan. DERIVED_PART_NUMBERS geleert. DigiKey-Stichwortsuche bevorzugt den Hersteller aus dem Schaltplan statt des billigsten Doppelgaengers. Netzliste identisch, ERC 0 Fehler. Stueckliste: 44 Positionen, alle eindeutig und lieferbar, 48,29 EUR. Task 0041 abgeschlossen; in Task 0042 zwei durch SHBS-17 erledigte Schritte vermerkt.

Co-Authored-By: Claude Opus 5.5 <noreply@anthropic.com>
Parts:
- J6: Manufacturer (none) -> Würth Elektronik; Manufacturer_Part_Number (none) -> 61200621621; Mouser Part Number (none) -> 710-61200621621
Changed lines of the file:
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@@
+			)
+		)
+		(property "Manufacturer" "Würth Elektronik"
+			(at 165.1 63.5 0)
+			(effects
+				(font
+					(size 1.27 1.27)
+				)
+				(hide yes)
+			)
+		)
+		(property "Manufacturer_Part_Number" "61200621621"
+			(at 165.1 63.5 0)
+			(effects
+				(font
+					(size 1.27 1.27)
+				)
+				(hide yes)
+			)
+		)
+		(property "Mouser Part Number" "710-61200621621"
+			(at 165.1 63.5 0)
+			(effects
+				(font
+					(size 1.27 1.27)
+				)
+				(hide yes)
 			)
 		)

Commit message: v0.00.001 fix(SHBS-16): D10-Verpolung behoben, LED-Symbole vereinheitlicht, FB1 und J6 bereinigt
Footprint WL-TMRC_3MM hatte Pad 1 = Anode, Device:LED hat Pin 1 = Kathode: D10 lag mit der Kathode an +3V3 und haette nie geleuchtet. Footprint auf Pad 1 = K / Pad 2 = A umnummeriert (wie WL-TMRW_3MM), Wuerth-Symbol mitgezogen. D7 von WL-TMRC_3MM auf Device:LED, so platziert, dass K/A auf den bisherigen Drahtenden liegen. FB1 auf Device:FerriteBead, J6-Wert auf 61200621621.

Gegenprobe: ERC 0 Fehler; Netzliste mit gleichen Bauteilen je Netz, nur D7-Pinnummern getauscht; Polaritaet aller vier LEDs auf Pad-Ebene geprueft. Beim naechsten PCB-Abgleich Footprint von D7/D10 aus der Bibliothek aktualisieren. Task 0042 abgeschlossen.

Co-Authored-By: Claude Opus 5.5 <noreply@anthropic.com>
Parts:
- D7: symbol WL-TMRC_3MM:WL-TMRC_3MM -> Device:LED
- J6: value Conn_02x03_Odd_Even -> 61200621621
Connections:
- net +3V3: now also D7.2 (A); no longer D7.1
- net at R13.2: now also D7.1 (K); no longer D7.2
Changed lines of the file:
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@@
 	)
 	(symbol
-		(lib_id "WL-TMRC_3MM:WL-TMRC_3MM")
-		(at 261.62 107.95 180)
+		(lib_id "Device:LED")
+		(at 262.89 107.95 0)
 		(unit 1)
 		(exclude_from_sim no)
@@
 			)
 		)
-		(property "Value" "Conn_02x03_Odd_Even"
+		(property "Value" "61200621621"
 			(at 166.37 57.15 0)
 			(effects

Commit message: v0.00.001 fix(SHBS-17): Q1-Q4 auf BC33740BU mit geraden Beinen, TA-Variante passte nicht auf TO-92_Inline
Die Gurt-Variante BC33740TA hat auf 2,54 mm aufgebogene Anschlussbeine, der Footprint TO-92_Inline hat 1,27 mm Raster. Umgestellt auf onsemi BC33740BU (gleiches Datenblatt, gerade Beine, Pinbelegung C-B-E unveraendert). Beim systematischen Footprint-Abgleich aufgefallen: alle anderen 72 Bauteile passen zu ihrem Footprint.

Gegenprobe: Netzliste identisch, Stueckliste 44 Positionen eindeutig und lieferbar.

Co-Authored-By: Claude Opus 5.5 <noreply@anthropic.com>
Parts:
- Q1, Q2, Q3, Q4: Manufacturer_Part_Number BC33740TA -> BC33740BU; Mouser Part Number 512-BC33740TA -> 512-BC33740BU
Changed lines of the file:
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@@
 			)
 		)
-		(property "Manufacturer_Part_Number" "BC33740TA"
+		(property "Manufacturer_Part_Number" "BC33740BU"
 			(at 246.38 148.59 0)
 			(effects
@@
 			)
 		)
-		(property "Mouser Part Number" "512-BC33740TA"
+		(property "Mouser Part Number" "512-BC33740BU"
 			(at 246.38 148.59 0)
 			(effects
@@
 			)
 		)
-		(property "Manufacturer_Part_Number" "BC33740TA"
+		(property "Manufacturer_Part_Number" "BC33740BU"
 			(at 219.71 104.14 0)
 			(effects
@@
 			)
 		)
-		(property "Mouser Part Number" "512-BC33740TA"
+		(property "Mouser Part Number" "512-BC33740BU"
 			(at 219.71 104.14 0)
 			(effects
@@
 			)
 		)
-		(property "Manufacturer_Part_Number" "BC33740TA"
+		(property "Manufacturer_Part_Number" "BC33740BU"
 			(at 228.6 118.11 0)
 			(effects
@@
 			)
 		)
-		(property "Mouser Part Number" "512-BC33740TA"
+		(property "Mouser Part Number" "512-BC33740BU"
 			(at 228.6 118.11 0)
 			(effects
@@
 			)
 		)
-		(property "Manufacturer_Part_Number" "BC33740TA"
+		(property "Manufacturer_Part_Number" "BC33740BU"
 			(at 238.76 133.35 0)
 			(effects
@@
 			)
 		)
-		(property "Mouser Part Number" "512-BC33740TA"
+		(property "Mouser Part Number" "512-BC33740BU"
 			(at 238.76 133.35 0)
 			(effects

Commit message: v0.00.001 feat(SHBS-25): Taster S2 auf liegenden C&K PTS645VL58-2 LFS umgestellt
Neuer Bauteilordner pcb/Bauteile/PTS645VL58-2LFS mit KiCad-Footprint und
Herstellermodell (kicad-packages3D), in fp-lib-table eingetragen. S2 im
Schaltplan: Footprint, Wert, Hersteller, Bestellnummern (Mouser
611-PTS645VL582, DigiKey CKN9116-ND); Altfelder des Bourns-Imports
bereinigt. Stücklisten-Generator kennt den neuen THT-Footprint,
Stückliste neu erzeugt. ERC unverändert.

Co-Authored-By: Claude Opus 5.5 <noreply@anthropic.com>
Parts:
- S2: value 1543-650-149 -> PTS645VL58-2 LFS; footprint 1543-650-149:1543650149 -> PTS645VL58-2LFS:SW_Tactile_SPST_Angled_PTS645Vx58-2LFS; ARROW_PART_NUMBER 1543-650-149 -> (none); ARROW_PRICE-STOCK https://www.arrow.com/en/products/1543-650-149/bourns -> (none); Availability In Stock -> (none); Check_prices https://www.snapeda.com/parts/1543-650-149/Bourns/view-part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 -> (none); DESCRIPTION Pushbutton Switches Push Switch -> Tactile switch SPST, right angle, 6 x 6 mm, actuator 5.8 mm; Description_1 Switch Push Button SPST Round Plunger 0.01A 24VAC 24VDC PC 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 -> Tactile switch SPST, right angle, 6 x 6 mm, actuator 5.8 mm; HEIGHT 15.1mm -> (none); MANUFACTURER (none) -> C&K; MANUFACTURER_NAME Bourns -> C&K; MANUFACTURER_PART_NUMBER 1543-650-149 -> PTS645VL58-2 LFS; MF Bourns -> C&K; MOUSER_PART_NUMBER 652-1543-650-149 -> 611-PTS645VL582; MOUSER_PRICE-STOCK https://www.mouser.co.uk/ProductDetail/Bourns/1543-650-149?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 -> https://www.mouser.de/ProductDetail/611-PTS645VL582; MP 1543-650-149 -> PTS645VL58-2 LFS; Purchase-URL https://www.snapeda.com/api/url_track_click_mouser/?unipart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 -> (none); SnapEDA_Link https://www.snapeda.com/parts/1543-650-149/Bourns/view-part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 -> (none)
Changed lines of the file:
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@@
 			)
 		)
-		(property "Value" "1543-650-149"
+		(property "Value" "PTS645VL58-2 LFS"
 			(at 30.48 54.6099 90)
 			(effects
@@
 			)
 		)
-		(property "Footprint" "1543-650-149:1543650149"
-			(at 24.13 63.5 0)
-			(effects
-				(font
-					(size 1.27 1.27)
-				)
-				(justify bottom)
-				(hide yes)
-			)
-		)
-		(property "Datasheet" ""
-			(at 24.13 63.5 0)
-			(effects
-				(font
-					(size 1.27 1.27)
-				)
-				(hide yes)
-			)
-		)
-		(property "Description" "Pushbutton Switches Push Switch"
-			(at 24.13 63.5 0)
-			(effects
-				(font
-					(size 1.27 1.27)
-				)
-				(hide yes)
-			)
-		)
-		(property "MANUFACTURER_NAME" "Bourns"
-			(at 24.13 63.5 0)
-			(effects
-				(font
-					(size 1.27 1.27)
-				)
-				(justify bottom)
-				(hide yes)
-			)
-		)
-		(property "MF" "Bourns"
-			(at 24.13 63.5 0)
-			(effects
-				(font
-					(size 1.27 1.27)
-				)
-				(justify bottom)
-				(hide yes)
-			)
-		)
-		(property "MOUSER_PRICE-STOCK" "https://www.mouser.co.uk/ProductDetail/Bourns/1543-650-149?qs=2f2kQrcl%2FoiIszYh%252BBIYwA%3D%3D"
-			(at 24.13 63.5 0)
-			(effects
-				(font
-					(size 1.27 1.27)
-				)
-				(justify bottom)
-				(hide yes)
-			)
-		)
-		(property "DESCRIPTION" "Pushbutton Switches Push Switch"
-			(at 24.13 63.5 0)
-			(effects
-				(font
-					(size 1.27 1.27)
-				)
-				(justify bottom)
-				(hide yes)
-			)
-		)
-		(property "MOUSER_PART_NUMBER" "652-1543-650-149"
+		(property "Footprint" "PTS645VL58-2LFS:SW_Tactile_SPST_Angled_PTS645Vx58-2LFS"
+			(at 24.13 63.5 0)
+			(effects
+				(font
+					(size 1.27 1.27)
+				)
+				(justify bottom)
+				(hide yes)
+			)
+		)
+		(property "Datasheet" "https://www.ckswitches.com/media/1471/pts645.pdf"
+			(at 24.13 63.5 0)
+			(effects
+				(font
+					(size 1.27 1.27)
+				)
+				(hide yes)
+			)
+		)
+		(property "Description" "Tactile switch SPST, right angle, 6 x 6 mm, actuator 5.8 mm"
+			(at 24.13 63.5 0)
+			(effects
+				(font
+					(size 1.27 1.27)
+				)
+				(hide yes)
+			)
+		)
+		(property "MANUFACTURER_NAME" "C&K"
+			(at 24.13 63.5 0)
+			(effects
+				(font
+					(size 1.27 1.27)
+				)
+				(justify bottom)
+				(hide yes)
+			)
+		)
+		(property "MF" "C&K"
+			(at 24.13 63.5 0)
+			(effects
+				(font
+					(size 1.27 1.27)
+				)
+				(justify bottom)
+				(hide yes)
+			)
+		)
+		(property "MOUSER_PRICE-STOCK" "https://www.mouser.de/ProductDetail/611-PTS645VL582"
+			(at 24.13 63.5 0)
+			(effects
+				(font
+					(size 1.27 1.27)
+				)
+				(justify bottom)
+				(hide yes)
+			)
+		)
+		(property "DESCRIPTION" "Tactile switch SPST, right angle, 6 x 6 mm, actuator 5.8 mm"
+			(at 24.13 63.5 0)
+			(effects
+				(font
+					(size 1.27 1.27)
+				)
+				(justify bottom)
+				(hide yes)
+			)
+		)
+		(property "MOUSER_PART_NUMBER" "611-PTS645VL582"
 			(at 24.13 63.5 0)
 			(effects
@@
 			)
 		)
-		(property "Check_prices" "https://www.snapeda.com/parts/1543-650-149/Bourns/view-part/?ref=eda"
-			(at 24.13 63.5 0)
-			(effects
-				(font
-					(size 1.27 1.27)
-				)
-				(justify bottom)
-				(hide yes)
-			)
-		)
-		(property "HEIGHT" "15.1mm"
-			(at 24.13 63.5 0)
-			(effects
-				(font
-					(size 1.27 1.27)
-				)
-				(justify bottom)
-				(hide yes)
-			)
-		)
-		(property "MP" "1543-650-149"
-			(at 24.13 63.5 0)
-			(effects
-				(font
-					(size 1.27 1.27)
-				)
-				(justify bottom)
-				(hide yes)
-			)
-		)
-		(property "SnapEDA_Link" "https://www.snapeda.com/parts/1543-650-149/Bourns/view-part/?ref=snap"
-			(at 24.13 63.5 0)
-			(effects
-				(font
-					(size 1.27 1.27)
-				)
-				(justify bottom)
-				(hide yes)
-			)
-		)
-		(property "ARROW_PRICE-STOCK" "https://www.arrow.com/en/products/1543-650-149/bourns"
-			(at 24.13 63.5 0)
-			(effects
-				(font
-					(size 1.27 1.27)
-				)
-				(justify bottom)
-				(hide yes)
-			)
-		)
-		(property "ARROW_PART_NUMBER" "1543-650-149"
-			(at 24.13 63.5 0)
-			(effects
-				(font
-					(size 1.27 1.27)
-				)
-				(justify bottom)
-				(hide yes)
-			)
-		)
-		(property "Purchase-URL" "https://www.snapeda.com/api/url_track_click_mouser/?unipart_id=2633736&manufacturer=Bourns&part_name=1543-650-149&search_term=1543-650-149"
-			(at 24.13 63.5 0)
-			(effects
-				(font
-					(size 1.27 1.27)
-				)
-				(justify bottom)
-				(hide yes)
-			)
-		)
-		(property "Description_1" "Switch Push Button SPST Round Plunger 0.01A 24VAC 24VDC PC Pins Thru-Hole"
-			(at 24.13 63.5 0)
-			(effects
-				(font
-					(size 1.27 1.27)
-				)
-				(justify bottom)
-				(hide yes)
-			)
-		)
-		(property "Availability" "In Stock"
-			(at 24.13 63.5 0)
-			(effects
-				(font
-					(size 1.27 1.27)
-				)
-				(justify bottom)
-				(hide yes)
-			)
-		)
-		(property "MANUFACTURER_PART_NUMBER" "1543-650-149"
-			(at 24.13 63.5 0)
-			(effects
-				(font
-					(size 1.27 1.27)
-				)
-				(justify bottom)
-				(hide yes)
-			)
-		)
-		(property "MANUFACTURER" ""
+		(property "Check_prices" ""
+			(at 24.13 63.5 0)
+			(effects
+				(font
+					(size 1.27 1.27)
+				)
+				(justify bottom)
+				(hide yes)
+			)
+		)
+		(property "HEIGHT" ""
+			(at 24.13 63.5 0)
+			(effects
+				(font
+					(size 1.27 1.27)
+				)
+				(justify bottom)
+				(hide yes)
+			)
+		)
+		(property "MP" "PTS645VL58-2 LFS"
+			(at 24.13 63.5 0)
+			(effects
+				(font
+					(size 1.27 1.27)
+				)
+				(justify bottom)
+				(hide yes)
+			)
+		)
+		(property "SnapEDA_Link" ""
+			(at 24.13 63.5 0)
+			(effects
+				(font
+					(size 1.27 1.27)
+				)
+				(justify bottom)
+				(hide yes)
+			)
+		)
+		(property "ARROW_PRICE-STOCK" ""
+			(at 24.13 63.5 0)
+			(effects
+				(font
+					(size 1.27 1.27)
+				)
+				(justify bottom)
+				(hide yes)
+			)
+		)
+		(property "ARROW_PART_NUMBER" ""
+			(at 24.13 63.5 0)
+			(effects
+				(font
+					(size 1.27 1.27)
+				)
+				(justify bottom)
+				(hide yes)
+			)
+		)
+		(property "Purchase-URL" ""
+			(at 24.13 63.5 0)
+			(effects
+				(font
+					(size 1.27 1.27)
+				)
+				(justify bottom)
+				(hide yes)
+			)
+		)
+		(property "Description_1" "Tactile switch SPST, right angle, 6 x 6 mm, actuator 5.8 mm"
+			(at 24.13 63.5 0)
+			(effects
+				(font
+					(size 1.27 1.27)
+				)
+				(justify bottom)
+				(hide yes)
+			)
+		)
+		(property "Availability" ""
+			(at 24.13 63.5 0)
+			(effects
+				(font
+					(size 1.27 1.27)
+				)
+				(justify bottom)
+				(hide yes)
+			)
+		)
+		(property "MANUFACTURER_PART_NUMBER" "PTS645VL58-2 LFS"
+			(at 24.13 63.5 0)
+			(effects
+				(font
+					(size 1.27 1.27)
+				)
+				(justify bottom)
+				(hide yes)
+			)
+		)
+		(property "MANUFACTURER" "C&K"
 			(at 24.13 63.5 90)
 			(effects

Commit message: v0.00.001 fix(SHBS-41): LED-Treiberstufe entfernt, Widerstände auf 0805, LEDs liegend
Q1-Q4 und R23-R26 entfallen, die LEDs hängen direkt am GPIO
(GPIO -> Vorwiderstand -> LED -> GND). R13-R16 und R9 als 0805,
R14 (blau) 100 Ohm. D7-D10 mit liegendem Footprint
LED_D3.0mm_Horizontal_O1.27mm_Z2.0mm. ERC 0/0.

Co-Authored-By: Claude Opus 5.5 <noreply@anthropic.com>
Parts:
- removed Q1, Q2, Q3, Q4: BC337, Package_TO_SOT_THT:TO-92_Inline, symbol Transistor_BJT:BC337
- removed R23, R24, R25, R26: 4,7k, Resistor_THT:R_Axial_DIN0617_L17.0mm_D6.0mm_P20.32mm_Horizontal, symbol Device:R
- D10, D7: footprint WL-TMRC_3MM:WL-TMRC_3MM -> LED_THT:LED_D3.0mm_Horizontal_O1.27mm_Z2.0mm
- D8, D9: footprint WL-TMRW_3MM:WL-TMRW_3MM -> LED_THT:LED_D3.0mm_Horizontal_O1.27mm_Z2.0mm
- R13, R15, R16: value 220 -> 220Ω; footprint Resistor_THT:R_Axial_DIN0617_L17.0mm_D6.0mm_P20.32mm_Horizontal -> Resistor_SMD:R_0805_2012Metric; Manufacturer Vishay BC Components -> YAGEO; Manufacturer_Part_Number PR02000202200JR500 -> RC0805FR-07220RL; Mouser Part Number 594-5083NW220R0J -> 603-RC0805FR-07220RL
- R14: value 220 -> 100Ω; footprint Resistor_THT:R_Axial_DIN0617_L17.0mm_D6.0mm_P20.32mm_Horizontal -> Resistor_SMD:R_0805_2012Metric; Manufacturer Vishay BC Components -> YAGEO; Manufacturer_Part_Number PR02000202200JR500 -> RC0805FR-07100RL; Mouser Part Number 594-5083NW220R0J -> 603-RC0805FR-07100RL
- R9: value 10k -> 10kΩ; footprint Resistor_THT:R_Axial_DIN0207_L6.3mm_D2.5mm_P10.16mm_Horizontal -> Resistor_SMD:R_0805_2012Metric; Manufacturer_Part_Number MFR-25FBF52-10K -> RC0805FR-0710KL; Mouser Part Number 603-MFR-25FBF52-10K -> 603-RC0805FR-0710KL
Connections:
- net +3V3: no longer D10.2 (A), D7.2 (A), D8.2 (A), D9.2 (A)
- net GND: now also D10.1 (K), D7.1 (K), D8.1 (K), D9.1 (K)
- net at R14.2: now also D8.2 (A)
- net at R15.2: now also D9.2 (A); no longer D9.1 (K)
- net at R13.2: now also D7.2 (A); no longer D7.1 (K)
- net at R14.1: now also U6.25 (GPIO48/SPICLK_N/SUBSPICLK_N_DIFF); no longer D8.1 (K)
- net at R13.1: now also U6.23 (GPIO21)
- net at R15.1: now also U6.31 (GPIO38/FSPIWP/SUBSPIWP)
- net at R16.2: now also D10.2 (A); no longer D10.1 (K)
- net at U6.24 (GPIO47/SPICLK_P/SUBSPICLK_P_DIFF): now also R16.1
Other:
- moved on the sheet: D10, D7, D8, D9, R13, R14, R15, R16
