File: pcb/BasisStation/Stromversorgung.kicad_sch (KiCad schematic)
At the start: 13 parts

Commit message: v0.00.001 feat(SHBS-17): USB-C-Buchse auf 12401598E4#2A umgestellt, Ersatz fuer PS1 vorgeschlagen
J1 und J_PWR1: Die abgekuendigte Amphenol 12401548E4#2A ist durch den
Nachfolger 12401598E4#2A ersetzt. Die neue Buchse ist nicht pad-kompatibel:
die B-Reihe ist SMD statt THT. Padbild aus dem Amphenol-STEP-Modell
ermittelt, es deckt sich mit dem KiCad-Footprint der Schwester
12401610E4-2A; uebernommen als shbs_power:USB_C_Receptacle_Amphenol_
12401598E4-2A. Schaltplan, Symbol-Cache und power.kicad_sym umgestellt,
ERC 0 Fehler.

PS1: Diodes AP3211KTR-G1 als pinkompatibler Ersatz fuer den MP2359
(NRND, ohne Lager) in der Stueckliste vorgeschlagen, Schaltplan noch
unveraendert. Alle 46 Positionen lieferbar, 47,78 EUR pro Baugruppe.

Co-Authored-By: Claude Opus 5.5 <noreply@anthropic.com>
Parts:
- J_PWR1: value 12401548E4-2A -> 12401598E4-2A; footprint shbs_power:USB_C_Receptacle_Amphenol_12401548E4-2A -> shbs_power:USB_C_Receptacle_Amphenol_12401598E4-2A; Manufacturer_Part_Number 12401548E4#2A -> 12401598E4#2A; Mouser Part Number 640-12401548E42A -> 523-12401598E4#2A; Notes Alternative: GCT USB4110-GF-A (verify land pattern before s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 -> Successor of discontinued 12401548E4#2A (SHBS-17); land pat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
Changed lines of the file:
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@@
 			)
 		)
-		(property "Value" "12401548E4-2A"
+		(property "Value" "12401598E4-2A"
 			(at 246.38 74.93 0)
 			(effects
@@
 			)
 		)
-		(property "Footprint" "shbs_power:USB_C_Receptacle_Amphenol_12401548E4-2A"
+		(property "Footprint" "shbs_power:USB_C_Receptacle_Amphenol_12401598E4-2A"
 			(at 246.38 83.82 0)
 			(effects
@@
 			)
 		)
-		(property "Description" "USB 2.0 Type-C receptacle, power (VBUS/CC), hybrid SMT+TH"
+		(property "Description" "USB 2.0 Type-C receptacle, power (VBUS/CC), SMT, shell through-hole"
 			(at 246.38 83.82 0)
 			(effects
@@
 			)
 		)
-		(property "Manufacturer_Part_Number" "12401548E4#2A"
+		(property "Manufacturer_Part_Number" "12401598E4#2A"
 			(at 246.38 83.82 0)
 			(effects
@@
 			)
 		)
-		(property "Mouser Part Number" "640-12401548E42A"
+		(property "Mouser Part Number" "523-12401598E4#2A"
 			(at 246.38 83.82 0)
 			(effects
@@
 			)
 		)
-		(property "Notes" "Alternative: GCT USB4110-GF-A (verify land pattern before swap)"
+		(property "Notes" "Successor of discontinued 12401548E4#2A (SHBS-17); land pattern checked against Amphenol STEP model"
 			(at 246.38 83.82 0)
 			(effects

Commit message: v0.00.001 feat(SHBS-17): PS1 auf AP3211 umgestellt, V_FB-Formel in der Doku korrigiert
Der MP2359 ist in allen Varianten NRND und ohne Lager. Ersetzt durch den
pinkompatiblen Diodes AP3211KTR-G1 (SOT-23-6, V_FB 0,81 V, 1,4 MHz,
asynchron, 1,5 A). Symbol in shbs_power:AP3211 umbenannt, Felder in
Schaltplan und power.kicad_sym umgestellt; Footprint MP2359DJ passt
unveraendert. ERC 0 Fehler, Netzliste an PS1 unveraendert. L1-Saettigung
(4,6 A) gegen Strombegrenzung (max. 2,4 A) geprueft.

power_supply.md: V_OUT-Formel nannte 0,6 V statt 0,81 V.

Co-Authored-By: Claude Opus 5.5 <noreply@anthropic.com>
Parts:
- PS1: value MP2359DJ -> AP3211; symbol shbs_power:MP2359DJ -> shbs_power:AP3211; Manufacturer Monolithic Power Systems -> Diodes Incorporated; Manufacturer_Part_Number MP2359DJ-LF-Z -> AP3211KTR-G1; Mouser Part Number 946-MP2359DJ-LF-Z -> 621-AP3211KTR-G1
Changed lines of the file:
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@@
 	)
 	(symbol
-		(lib_id "shbs_power:MP2359DJ")
+		(lib_id "shbs_power:AP3211")
 		(at 148.59 86.36 0)
 		(unit 1)
@@
 			)
 		)
-		(property "Value" "MP2359DJ"
+		(property "Value" "AP3211"
 			(at 148.59 78.74 0)
 			(effects
@@
 			)
 		)
-		(property "Datasheet" "https://www.monolithicpower.com/en/documentview/productdocument/index/version/2/document_type/Datasheet/lang/en/sku/MP2359/document_id/90"
+		(property "Datasheet" "https://www.diodes.com/assets/Datasheets/AP3211.pdf"
 			(at 148.59 86.36 0)
 			(effects
@@
 			)
 		)
-		(property "Description" "1.2A, 24V, 1.4MHz step-down converter, SOT23-6"
+		(property "Description" "1.5A, 18V, 1.4MHz asynchronous step-down converter, SOT-23-6 (pin-compatible successor of MP2359DJ, SHBS-17)"
 			(at 148.59 86.36 0)
 			(effects
@@
 			)
 		)
-		(property "Manufacturer" "Monolithic Power Systems"
+		(property "Manufacturer" "Diodes Incorporated"
 			(at 148.59 86.36 0)
 			(effects
@@
 			)
 		)
-		(property "Manufacturer_Part_Number" "MP2359DJ-LF-Z"
+		(property "Manufacturer_Part_Number" "AP3211KTR-G1"
 			(at 148.59 86.36 0)
 			(effects
@@
 			)
 		)
-		(property "Mouser Part Number" "946-MP2359DJ-LF-Z"
+		(property "Mouser Part Number" "621-AP3211KTR-G1"
 			(at 148.59 86.36 0)
 			(effects

Commit message: v0.00.001 feat(SHBS-17): Teilenummern fuer 29 Positionen in den Schaltplan uebernommen
Die vom Bediener freigegebenen Teilevorschlaege (Hausstandard Passivteile, LEDs, Q1-Q4, F1, FB1) stehen jetzt als Felder Manufacturer, Manufacturer_Part_Number und Mouser Part Number an 58 Instanzen. F1-Wert von Fuse auf 1.1A gesetzt. Gegenprobe: keine Felder verloren, Netzliste identisch (102 Netze), ERC 0 Fehler.

Stueckliste gruppiert jetzt nach Herstellerteilenummer (Werte sind uneinheitlich geschrieben): 44 Positionen, alle lieferbar, 47,78 EUR. PROPOSED_PARTS geleert, Hausstandard in hardware.md dokumentiert, Bestellteile in power_supply.md aktualisiert.

Co-Authored-By: Claude Opus 5.5 <noreply@anthropic.com>
Parts:
- C13: Manufacturer (none) -> Samsung; Manufacturer_Part_Number (none) -> CL21B106KOQNNNE; Mouser Part Number (none) -> 187-CL21B106KOQNNNE
- C14: Manufacturer (none) -> Samsung; Manufacturer_Part_Number (none) -> CL21A226MOQNNNE; Mouser Part Number (none) -> 187-CL21A226MOQNNNE
- C15: Manufacturer (none) -> YAGEO; Manufacturer_Part_Number (none) -> CC0805KRX7R9BB104; Mouser Part Number (none) -> 603-CC805KRX7R9BB104
- F1: value Fuse -> 1.1A; Manufacturer (none) -> Bourns; Manufacturer_Part_Number (none) -> MF-NSMF110-2; Mouser Part Number (none) -> 652-MF-NSMF110-2
- R17: Manufacturer (none) -> YAGEO; Manufacturer_Part_Number (none) -> RC0805FR-0749K9L; Mouser Part Number (none) -> 603-RC0805FR-0749K9L
- R18: Manufacturer (none) -> YAGEO; Manufacturer_Part_Number (none) -> RC0805FR-0716K2L; Mouser Part Number (none) -> 603-RC0805FR-0716K2L
- R19, R20: Manufacturer (none) -> YAGEO; Manufacturer_Part_Number (none) -> RC0805FR-075K1L; Mouser Part Number (none) -> 603-RC0805FR-075K1L
Changed lines of the file:
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@@
+			)
+		)
+		(property "Manufacturer" "YAGEO"
+			(at 231.14 95.25 0)
+			(effects
+				(font
+					(size 1.27 1.27)
+				)
+				(hide yes)
+			)
+		)
+		(property "Manufacturer_Part_Number" "RC0805FR-075K1L"
+			(at 231.14 95.25 0)
+			(effects
+				(font
+					(size 1.27 1.27)
+				)
+				(hide yes)
+			)
+		)
+		(property "Mouser Part Number" "603-RC0805FR-075K1L"
+			(at 231.14 95.25 0)
+			(effects
+				(font
+					(size 1.27 1.27)
+				)
+				(hide yes)
 			)
 		)
@@
 			)
 		)
+		(property "Manufacturer" "Samsung"
+			(at 167.64 68.58 0)
+			(effects
+				(font
+					(size 1.27 1.27)
+				)
+				(hide yes)
+			)
+		)
+		(property "Manufacturer_Part_Number" "CL21B106KOQNNNE"
+			(at 167.64 68.58 0)
+			(effects
+				(font
+					(size 1.27 1.27)
+				)
+				(hide yes)
+			)
+		)
+		(property "Mouser Part Number" "187-CL21B106KOQNNNE"
+			(at 167.64 68.58 0)
+			(effects
+				(font
+					(size 1.27 1.27)
+				)
+				(hide yes)
+			)
+		)
 		(pin "1"
 		)
@@
 			)
 		)
-		(property "Value" "Fuse"
+		(property "Value" "1.1A"
 			(at 203.2 80.01 90)
 			(effects
@@
 		(property "STANDARD" ""
 			(at 203.2 83.82 90)
+			(effects
+				(font
+					(size 1.27 1.27)
+				)
+				(hide yes)
+			)
+		)
+		(property "Manufacturer" "Bourns"
+			(at 203.2 83.82 0)
+			(effects
+				(font
+					(size 1.27 1.27)
+				)
+				(hide yes)
+			)
+		)
+		(property "Manufacturer_Part_Number" "MF-NSMF110-2"
+			(at 203.2 83.82 0)
+			(effects
+				(font
+					(size 1.27 1.27)
+				)
+				(hide yes)
+			)
+		)
+		(property "Mouser Part Number" "652-MF-NSMF110-2"
+			(at 203.2 83.82 0)
 			(effects
 				(font
@@
 			)
 		)
+		(property "Manufacturer" "YAGEO"
+			(at 111.76 97.79 0)
+			(effects
+				(font
+					(size 1.27 1.27)
+				)
+				(hide yes)
+			)
+		)
+		(property "Manufacturer_Part_Number" "RC0805FR-0716K2L"
+			(at 111.76 97.79 0)
+			(effects
+				(font
+					(size 1.27 1.27)
+				)
+				(hide yes)
+			)
+		)
+		(property "Mouser Part Number" "603-RC0805FR-0716K2L"
+			(at 111.76 97.79 0)
+			(effects
+				(font
+					(size 1.27 1.27)
+				)
+				(hide yes)
+			)
+		)
 		(pin "1"
 		)
@@
 			)
 		)
+		(property "Manufacturer" "Samsung"
+			(at 189.23 127 0)
+			(effects
+				(font
+					(size 1.27 1.27)
+				)
+				(hide yes)
+			)
+		)
+		(property "Manufacturer_Part_Number" "CL21A226MOQNNNE"
+			(at 189.23 127 0)
+			(effects
+				(font
+					(size 1.27 1.27)
+				)
+				(hide yes)
+			)
+		)
+		(property "Mouser Part Number" "187-CL21A226MOQNNNE"
+			(at 189.23 127 0)
+			(effects
+				(font
+					(size 1.27 1.27)
+				)
+				(hide yes)
+			)
+		)
 		(pin "1"
 		)
@@
 			)
 		)
+		(property "Manufacturer" "YAGEO"
+			(at 147.32 116.84 0)
+			(effects
+				(font
+					(size 1.27 1.27)
+				)
+				(hide yes)
+			)
+		)
+		(property "Manufacturer_Part_Number" "CC0805KRX7R9BB104"
+			(at 147.32 116.84 0)
+			(effects
+				(font
+					(size 1.27 1.27)
+				)
+				(hide yes)
+			)
+		)
+		(property "Mouser Part Number" "603-CC805KRX7R9BB104"
+			(at 147.32 116.84 0)
+			(effects
+				(font
+					(size 1.27 1.27)
+				)
+				(hide yes)
+			)
+		)
 		(pin "1"
 		)
@@
 			)
 		)
+		(property "Manufacturer" "YAGEO"
+			(at 124.46 97.79 0)
+			(effects
+				(font
+					(size 1.27 1.27)
+				)
+				(hide yes)
+			)
+		)
+		(property "Manufacturer_Part_Number" "RC0805FR-0749K9L"
+			(at 124.46 97.79 0)
+			(effects
+				(font
+					(size 1.27 1.27)
+				)
+				(hide yes)
+			)
+		)
+		(property "Mouser Part Number" "603-RC0805FR-0749K9L"
+			(at 124.46 97.79 0)
+			(effects
+				(font
+					(size 1.27 1.27)
+				)
+				(hide yes)
+			)
+		)
 		(pin "1"
 		)
@@
 			(at 219.71 95.25 0)
 			(effects
+				(font
+					(size 1.27 1.27)
+				)
+				(hide yes)
+			)
+		)
+		(property "Manufacturer" "YAGEO"
+			(at 219.71 95.25 0)
+			(effects
+				(font
+					(size 1.27 1.27)
+				)
+				(hide yes)
+			)
+		)
+		(property "Manufacturer_Part_Number" "RC0805FR-075K1L"
+			(at 219.71 95.25 0)
+			(effects
+				(font
+					(size 1.27 1.27)
+				)
+				(hide yes)
+			)
+		)
+		(property "Mouser Part Number" "603-RC0805FR-075K1L"
+			(at 219.71 95.25 0)
+			(effects

Commit message: v0.00.001 feat(SHBS-17): Abgeleitete Teilenummern bestaetigt und eingetragen, SHBS-17 abgeschlossen
D11 Comchip SS34-HF (SMA; die guenstigere Slkormicro-SS34 ist SMC und passt nicht auf D_SMA), D12 Littelfuse SMAJ5.0A, U1 D3V3XA4B10LP-7, L1 Bourns SRN6045TA-100M, J6 Wuerth 61200621621 als Felder im Schaltplan. DERIVED_PART_NUMBERS geleert. DigiKey-Stichwortsuche bevorzugt den Hersteller aus dem Schaltplan statt des billigsten Doppelgaengers. Netzliste identisch, ERC 0 Fehler. Stueckliste: 44 Positionen, alle eindeutig und lieferbar, 48,29 EUR. Task 0041 abgeschlossen; in Task 0042 zwei durch SHBS-17 erledigte Schritte vermerkt.

Co-Authored-By: Claude Opus 5.5 <noreply@anthropic.com>
Parts:
- D11: Manufacturer (none) -> Comchip Technology; Manufacturer_Part_Number (none) -> SS34-HF; Mouser Part Number (none) -> 750-SS34-HF
- D12: Manufacturer (none) -> Littelfuse; Manufacturer_Part_Number (none) -> SMAJ5.0A; Mouser Part Number (none) -> 576-SMAJ5.0A
- L1: Manufacturer (none) -> Bourns; Manufacturer_Part_Number (none) -> SRN6045TA-100M; Mouser Part Number (none) -> 652-SRN6045TA-100M
Changed lines of the file:
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@@
+			)
+		)
+		(property "Manufacturer" "Comchip Technology"
+			(at 165.1 116.84 0)
+			(effects
+				(font
+					(size 1.27 1.27)
+				)
+				(hide yes)
+			)
+		)
+		(property "Manufacturer_Part_Number" "SS34-HF"
+			(at 165.1 116.84 0)
+			(effects
+				(font
+					(size 1.27 1.27)
+				)
+				(hide yes)
+			)
+		)
+		(property "Mouser Part Number" "750-SS34-HF"
+			(at 165.1 116.84 0)
+			(effects
+				(font
+					(size 1.27 1.27)
+				)
+				(hide yes)
 			)
 		)
@@
 			)
 		)
+		(property "Manufacturer" "Littelfuse"
+			(at 182.88 68.58 0)
+			(effects
+				(font
+					(size 1.27 1.27)
+				)
+				(hide yes)
+			)
+		)
+		(property "Manufacturer_Part_Number" "SMAJ5.0A"
+			(at 182.88 68.58 0)
+			(effects
+				(font
+					(size 1.27 1.27)
+				)
+				(hide yes)
+			)
+		)
+		(property "Mouser Part Number" "576-SMAJ5.0A"
+			(at 182.88 68.58 0)
+			(effects
+				(font
+					(size 1.27 1.27)
+				)
+				(hide yes)
+			)
+		)
 		(pin "1"
 		)
@@
 			(effects
 				(font
+					(size 1.27 1.27)
+				)
+				(hide yes)
+			)
+		)
+		(property "Manufacturer" "Bourns"
+			(at 181.61 113.03 0)
+			(effects
+				(font
+					(size 1.27 1.27)
+				)
+				(hide yes)
+			)
+		)
+		(property "Manufacturer_Part_Number" "SRN6045TA-100M"
+			(at 181.61 113.03 0)
+			(effects
+				(font
+					(size 1.27 1.27)
+				)
+				(hide yes)
+			)
+		)
+		(property "Mouser Part Number" "652-SRN6045TA-100M"
+			(at 181.61 113.03 0)
+			(effects
+				(font
