File: pcb/BasisStation/Stromversorgung.kicad_sch (KiCad schematic)
At the start: 13 parts

Commit message: v0.00.001 fix(SHBS-20): USB-C J_PWR1 um VBUS-Pins B4/B9 und GND-Pins A12/B12 ergänzt
Das Symbol shbs_power:USB_C_Receptacle_Power führte nur A1/B1/A4/A9, die
Pads B4/B9/A12/B12 lagen ohne Netz. Die vier Pins sind jetzt unsichtbar
und als passive auf A4/A9 bzw. A1/B1 gestapelt (kein versteckter
power_in). Symbol-Cache im Schaltplan nachgezogen, power_supply.md
aktualisiert. PCB-Anbindung der Pads siehe c2ccc4a.

Co-Authored-By: Claude Opus 5.5 <noreply@anthropic.com>
Connections:
- net GND: now also J_PWR1.A12 (GND), J_PWR1.B12 (GND)
- net VBUS: now also J_PWR1.B4 (VBUS), J_PWR1.B9 (VBUS)
Changed lines of the file:
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@@
 		)
 	)
-	(label "VBUS"
-		(at 231.14 78.74 0)
+	(label "+5V"
+		(at 161.29 77.47 90)
 		(effects
 			(font
@@
 		)
 	)
-	(label "+5V"
-		(at 161.29 77.47 90)
+	(label "VBUS"
+		(at 231.14 78.74 0)
 		(effects
 			(font

Commit message: v0.00.001 (WIP) feat(SHBS-21): Netzklasse Power, Label SW und Session-Übergabe
Netzklasse Power (0,6 mm, Via 0,8/0,4) mit Mustern für VBUS, +5V, SW,
+3V3 und GND. Schaltknoten im Schaltplan als lokales Label SW benannt,
PCB per F8 nachgezogen. power_supply.md ergänzt. tmp/memory.md hält den
Session-Stand für die Weiterarbeit auf einem anderen Rechner fest
(nächster Schritt: Buck-Wandler kompakt platzieren).

Co-Authored-By: Claude Opus 5.5 <noreply@anthropic.com>
Connections:
- net SW: now reaches C15.2, D11.1 (K), L1.2, PS1.6 (SW)
Changed lines of the file:
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@@
+		)
+	)
+	(label "SW"
+		(at 163.83 86.36 0)
+		(effects
+			(font
+				(size 1.27 1.27)
+			)
+			(justify left bottom)
 		)
 	)
